File: ESP01_WLED.kicad_sch (KiCad schematic)
At the start: 10 parts, among them J2 Conn_01x02_Pin, U1 ESP-01v090, U2 AMS1117-3.3

Commit message: usb c
Parts:
- removed J2: Conn_01x02_Pin, Connector_PinHeader_2.54mm:PinHeader_1x02_P2.54mm_Vertical, symbol Connector:Conn_01x02_Pin
- added J3: USB_C_Receptacle_PowerOnly_6P, Connector_USB:USB_C_Receptacle_GCT_USB4125-xx-x_6P_TopMnt_Horizontal, symbol Connector:USB_C_Receptacle_PowerOnly_6P
- added R5, R6: 5.1k, Resistor_SMD:R_0805_2012Metric_Pad1.20x1.40mm_HandSolder, symbol Device:R_Small
Connections:
- net +5V: now also J3.A9 (VBUS), J3.B9 (VBUS)
- net GND: now also J3.A12 (GND), J3.B12 (GND), J3.S1 (SHIELD), R5.2, R6.2
- new net: J3.A5 (CC1), R5.1
- new net: J3.B5 (CC2), R6.1
