File: ESP01_WLED.kicad_pcb (KiCad board)
At the start: 2 copper layers, 14 x 26 mm, 17 parts, among them J2 Conn_01x02_Pin, U1 ESP-01v090, U1_ PinSocket_2x04_P2.54mm_Vertic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, U2 AMS1117-3.3

Commit message: usb c
Parts:
- removed J2: Conn_01x02_Pin, Connector_PinHeader_2.54mm:PinHeader_1x02_P2.54mm_Vertical
- added J3: USB_C_Receptacle_PowerOnly_6P, Connector_USB:USB_C_Receptacle_GCT_USB4125-xx-x_6P_TopMnt_Horizontal, F.Cu at (12.0, 13.0)
- added R5: 5.1k, Resistor_SMD:R_0805_2012Metric_Pad1.20x1.40mm_HandSolder, B.Cu at (10.0, 14.0)
- added R6: 5.1k, Resistor_SMD:R_0805_2012Metric_Pad1.20x1.40mm_HandSolder, B.Cu at (10.0, 12.0)
- C1, C2, R1, R2, U2: moved to B.Cu
- moved R4 9.00 mm to (4.00, 7.00), turned to 90 degrees
- moved C1 6.50 mm to (1.50, 4.00), turned to -90 degrees
- moved C2 6.50 mm to (12.5, 4.00), turned to -90 degrees
- moved R3 6.10 mm to (6.50, 7.00), turned to 90 degrees
- moved R2 4.30 mm to (6.50, 11.5), turned to -90 degrees
- moved R1 3.54 mm to (6.50, 15.5), turned to -90 degrees
- moved J1 3.00 mm to (4.00, 15.5)
Connections:
- U1_ pad 1: (no net) -> unconnected-(U1-URXD-Pad8)
- U1_ pad 8: (no net) -> unconnected-(U1-UTXD-Pad1)
Routing:
- net GND: track 3.53 -> 15.2 mm
- net Net-(U1-GPIO0): track 5.78 -> 13.2 mm
- net +5V: track 16.1 -> 22.5 mm
- net 3V3: track 40.6 -> 46.9 mm, vias 0 -> 2
- net Net-(U1-RST): track 10.4 -> 7.42 mm, vias 1 -> 0
- net Net-(U1-GPIO2): track 10.6 -> 13.5 mm, vias 0 -> 1
- net Net-(J3-CC2): vias 0 -> 1
- net Net-(J3-CC1): vias 0 -> 1
- added copper zone on B.Cu, net GND
- added copper zone on F.Cu, net GND
