File: ESP01_WLED_pannel.kicad_pcb (KiCad board)
At the start: 2 copper layers, 94 x 96 mm, 648 parts, among them J2 Conn_01x02_Pin, U1 ESP-01v090, U1_ PinSocket_2x04_P2.54mm_Vertic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, U2 AMS1117-3.3

Commit message: usb c
Parts:
- removed the C1 at (121.5, 65.0)
- removed the C1 at (169.5, 93.0)
- removed the C1 at (185.5, 65.0)
- removed the C1 at (153.5, 37.0)
- removed the C1 at (121.5, 93.0)
- removed the C1 at (121.5, 37.0)
- removed the C1 at (153.5, 93.0)
- removed the C1 at (153.5, 65.0)
- removed the C1 at (169.5, 37.0)
- removed the C1 at (137.5, 93.0)
- removed the C1 at (169.5, 65.0)
- removed the C1 at (105.5, 65.0)
- removed the C1 at (105.5, 93.0)
- removed the C1 at (185.5, 37.0)
- removed the C1 at (105.5, 37.0)
- removed the C1 at (185.5, 93.0)
- removed the C1 at (137.5, 65.0)
- removed the C1 at (137.5, 37.0)
- removed the C2 at (111.5, 65.0)
- removed the C2 at (159.5, 65.0)
- removed the C2 at (127.5, 37.0)
- removed the C2 at (111.5, 93.0)
- removed the C2 at (175.5, 37.0)
- removed the C2 at (143.5, 65.0)
- removed the C2 at (191.5, 37.0)
- removed the C2 at (143.5, 37.0)
- removed the C2 at (159.5, 37.0)
- removed the C2 at (175.5, 93.0)
- removed the C2 at (191.5, 93.0)
- removed the C2 at (175.5, 65.0)
- removed the C2 at (159.5, 93.0)
- removed the C2 at (191.5, 65.0)
- removed the C2 at (127.5, 65.0)
- removed the C2 at (111.5, 37.0)
- removed the C2 at (127.5, 93.0)
- removed the C2 at (143.5, 93.0)
- removed the J1 at (140.5, 70.5)
- removed the J1 at (188.5, 70.5)
- removed the J1 at (124.5, 70.5)
- removed the J1 at (156.5, 70.5)
- removed the J1 at (124.5, 98.5)
- removed the J1 at (124.5, 42.5)
- removed the J1 at (188.5, 98.5)
- removed the J1 at (108.5, 70.5)
- removed the J1 at (140.5, 98.5)
- removed the J1 at (108.5, 42.5)
- removed the J1 at (172.5, 42.5)
- removed the J1 at (172.5, 98.5)
- removed the J1 at (156.5, 98.5)
- removed the J1 at (156.5, 42.5)
- removed the J1 at (140.5, 42.5)
- removed the J1 at (172.5, 70.5)
- removed the J1 at (188.5, 42.5)
- removed the J1 at (108.5, 98.5)
- removed J2 (x18): Conn_01x02_Pin, Connector_PinHeader_2.54mm:PinHeader_1x02_P2.54mm_Vertical
- removed KiKit_MB_11_5, KiKit_MB_12_5, KiKit_MB_13_5, KiKit_MB_14_5, KiKit_MB_17_5, KiKit_MB_18_5, KiKit_MB_19_5, KiKit_MB_1_5, KiKit_MB_20_5, KiKit_MB_23_5, KiKit_MB_24_5, KiKit_MB_25_5, KiKit_MB_26_5, KiKit_MB_29_5, KiKit_MB_2_5, KiKit_MB_30_5, KiKit_MB_33_5, KiKit_MB_34_5, KiKit_MB_37_5, KiKit_MB_38_5, KiKit_MB_39_5, KiKit_MB_40_5, KiKit_MB_43_5, KiKit_MB_44_5, KiKit_MB_45_5, KiKit_MB_46_5, KiKit_MB_49_5, KiKit_MB_50_5, KiKit_MB_51_5, KiKit_MB_52_5, KiKit_MB_55_5, KiKit_MB_56_5, KiKit_MB_57_5, KiKit_MB_58_5, KiKit_MB_5_5, KiKit_MB_61_5, KiKit_MB_62_5, KiKit_MB_65_5, KiKit_MB_66_5, KiKit_MB_69_5, KiKit_MB_6_5, KiKit_MB_70_5, KiKit_MB_71_5, KiKit_MB_72_5, KiKit_MB_75_5, KiKit_MB_76_5, KiKit_MB_77_5, KiKit_MB_78_5, KiKit_MB_7_5, KiKit_MB_81_5, KiKit_MB_82_5, KiKit_MB_83_5, KiKit_MB_84_5, KiKit_MB_87_5, KiKit_MB_88_5, KiKit_MB_89_5, KiKit_MB_8_5, KiKit_MB_90_5, KiKit_MB_93_5, KiKit_MB_94_5: NPTH, NPTH
- removed the R1 at (143.5, 43.0)
- removed the R1 at (143.5, 71.0)
- removed the R1 at (175.5, 99.0)
- removed the R1 at (111.5, 43.0)
- removed the R1 at (159.5, 99.0)
- removed the R1 at (159.5, 71.0)
- removed the R1 at (159.5, 43.0)
- removed the R1 at (127.5, 99.0)
- removed the R1 at (127.5, 43.0)
- removed the R1 at (111.5, 99.0)
- removed the R1 at (127.5, 71.0)
- removed the R1 at (191.5, 99.0)
- removed the R1 at (191.5, 43.0)
- removed the R1 at (175.5, 43.0)
- removed the R1 at (191.5, 71.0)
- removed the R1 at (111.5, 71.0)
- removed the R1 at (143.5, 99.0)
- removed the R1 at (175.5, 71.0)
- removed the R2 at (175.5, 69.0)
- removed the R2 at (159.5, 41.0)
- removed the R2 at (159.5, 97.0)
- removed the R2 at (143.5, 41.0)
- removed the R2 at (191.5, 97.0)
- removed the R2 at (191.5, 69.0)
- removed the R2 at (111.5, 69.0)
- removed the R2 at (175.5, 41.0)
- removed the R2 at (191.5, 41.0)
- removed the R2 at (127.5, 69.0)
- removed the R2 at (111.5, 97.0)
- removed the R2 at (143.5, 69.0)
- removed the R2 at (175.5, 97.0)
- removed the R2 at (127.5, 41.0)
- removed the R2 at (127.5, 97.0)
- removed the R2 at (143.5, 97.0)
- removed the R2 at (159.5, 69.0)
- removed the R2 at (111.5, 41.0)
- removed the R3 at (175.5, 67.0)
- removed the R3 at (175.5, 39.0)
- removed the R3 at (175.5, 95.0)
- removed the R3 at (191.5, 95.0)
- removed the R3 at (143.5, 39.0)
- removed the R3 at (159.5, 95.0)
- removed the R3 at (127.5, 95.0)
- removed the R3 at (127.5, 67.0)
- removed the R3 at (111.5, 39.0)
- removed the R3 at (111.5, 67.0)
- removed the R3 at (159.5, 67.0)
- removed the R3 at (143.5, 67.0)
- removed the R3 at (111.5, 95.0)
- removed the R3 at (143.5, 95.0)
- removed the R3 at (191.5, 67.0)
- removed the R3 at (127.5, 39.0)
- removed the R3 at (191.5, 39.0)
- removed the R3 at (159.5, 39.0)
- removed the R4 at (169.5, 71.0)
- removed the R4 at (137.5, 71.0)
- removed the R4 at (105.5, 99.0)
- removed the R4 at (185.5, 43.0)
- removed the R4 at (121.5, 99.0)
- removed the R4 at (121.5, 43.0)
- removed the R4 at (169.5, 99.0)
- removed the R4 at (153.5, 43.0)
- removed the R4 at (137.5, 99.0)
- removed the R4 at (105.5, 71.0)
- removed the R4 at (185.5, 71.0)
- removed the R4 at (185.5, 99.0)
- removed the R4 at (137.5, 43.0)
- removed the R4 at (105.5, 43.0)
- removed the R4 at (121.5, 71.0)
- removed the R4 at (169.5, 43.0)
- removed the R4 at (153.5, 71.0)
- removed the R4 at (153.5, 99.0)
- added C1: 22uF, Capacitor_SMD:C_0805_2012Metric_Pad1.18x1.45mm_HandSolder, B.Cu at (167.0, 87.0)
- added C1: 22uF, Capacitor_SMD:C_0805_2012Metric_Pad1.18x1.45mm_HandSolder, B.Cu at (183.0, 31.0)
- added C1: 22uF, Capacitor_SMD:C_0805_2012Metric_Pad1.18x1.45mm_HandSolder, B.Cu at (167.0, 59.0)
- added C1: 22uF, Capacitor_SMD:C_0805_2012Metric_Pad1.18x1.45mm_HandSolder, B.Cu at (183.0, 87.0)
- added C1: 22uF, Capacitor_SMD:C_0805_2012Metric_Pad1.18x1.45mm_HandSolder, B.Cu at (119.0, 87.0)
- added C1: 22uF, Capacitor_SMD:C_0805_2012Metric_Pad1.18x1.45mm_HandSolder, B.Cu at (103.0, 31.0)
- added C1: 22uF, Capacitor_SMD:C_0805_2012Metric_Pad1.18x1.45mm_HandSolder, B.Cu at (151.0, 87.0)
- added C1: 22uF, Capacitor_SMD:C_0805_2012Metric_Pad1.18x1.45mm_HandSolder, B.Cu at (135.0, 31.0)
- added C1: 22uF, Capacitor_SMD:C_0805_2012Metric_Pad1.18x1.45mm_HandSolder, B.Cu at (183.0, 59.0)
- added C1: 22uF, Capacitor_SMD:C_0805_2012Metric_Pad1.18x1.45mm_HandSolder, B.Cu at (167.0, 31.0)
- added C1: 22uF, Capacitor_SMD:C_0805_2012Metric_Pad1.18x1.45mm_HandSolder, B.Cu at (135.0, 87.0)
- added C1: 22uF, Capacitor_SMD:C_0805_2012Metric_Pad1.18x1.45mm_HandSolder, B.Cu at (119.0, 31.0)
- added C1: 22uF, Capacitor_SMD:C_0805_2012Metric_Pad1.18x1.45mm_HandSolder, B.Cu at (119.0, 59.0)
- added C1: 22uF, Capacitor_SMD:C_0805_2012Metric_Pad1.18x1.45mm_HandSolder, B.Cu at (151.0, 59.0)
- added C1: 22uF, Capacitor_SMD:C_0805_2012Metric_Pad1.18x1.45mm_HandSolder, B.Cu at (103.0, 59.0)
- added C1: 22uF, Capacitor_SMD:C_0805_2012Metric_Pad1.18x1.45mm_HandSolder, B.Cu at (135.0, 59.0)
- added C1: 22uF, Capacitor_SMD:C_0805_2012Metric_Pad1.18x1.45mm_HandSolder, B.Cu at (103.0, 87.0)
- added C1: 22uF, Capacitor_SMD:C_0805_2012Metric_Pad1.18x1.45mm_HandSolder, B.Cu at (151.0, 31.0)
- added C2: 22uF, Capacitor_SMD:C_0805_2012Metric_Pad1.18x1.45mm_HandSolder, B.Cu at (114.0, 87.0)
- added C2: 22uF, Capacitor_SMD:C_0805_2012Metric_Pad1.18x1.45mm_HandSolder, B.Cu at (146.0, 87.0)
- added C2: 22uF, Capacitor_SMD:C_0805_2012Metric_Pad1.18x1.45mm_HandSolder, B.Cu at (178.0, 31.0)
- added C2: 22uF, Capacitor_SMD:C_0805_2012Metric_Pad1.18x1.45mm_HandSolder, B.Cu at (162.0, 31.0)
- added C2: 22uF, Capacitor_SMD:C_0805_2012Metric_Pad1.18x1.45mm_HandSolder, B.Cu at (194.0, 59.0)
- added C2: 22uF, Capacitor_SMD:C_0805_2012Metric_Pad1.18x1.45mm_HandSolder, B.Cu at (130.0, 87.0)
- added C2: 22uF, Capacitor_SMD:C_0805_2012Metric_Pad1.18x1.45mm_HandSolder, B.Cu at (114.0, 59.0)
- added C2: 22uF, Capacitor_SMD:C_0805_2012Metric_Pad1.18x1.45mm_HandSolder, B.Cu at (130.0, 31.0)
- added C2: 22uF, Capacitor_SMD:C_0805_2012Metric_Pad1.18x1.45mm_HandSolder, B.Cu at (130.0, 59.0)
- added C2: 22uF, Capacitor_SMD:C_0805_2012Metric_Pad1.18x1.45mm_HandSolder, B.Cu at (162.0, 87.0)
- added C2: 22uF, Capacitor_SMD:C_0805_2012Metric_Pad1.18x1.45mm_HandSolder, B.Cu at (162.0, 59.0)
- added C2: 22uF, Capacitor_SMD:C_0805_2012Metric_Pad1.18x1.45mm_HandSolder, B.Cu at (146.0, 31.0)
- added C2: 22uF, Capacitor_SMD:C_0805_2012Metric_Pad1.18x1.45mm_HandSolder, B.Cu at (114.0, 31.0)
- added C2: 22uF, Capacitor_SMD:C_0805_2012Metric_Pad1.18x1.45mm_HandSolder, B.Cu at (194.0, 31.0)
- added C2: 22uF, Capacitor_SMD:C_0805_2012Metric_Pad1.18x1.45mm_HandSolder, B.Cu at (146.0, 59.0)
- added C2: 22uF, Capacitor_SMD:C_0805_2012Metric_Pad1.18x1.45mm_HandSolder, B.Cu at (178.0, 59.0)
- added C2: 22uF, Capacitor_SMD:C_0805_2012Metric_Pad1.18x1.45mm_HandSolder, B.Cu at (194.0, 87.0)
- added C2: 22uF, Capacitor_SMD:C_0805_2012Metric_Pad1.18x1.45mm_HandSolder, B.Cu at (178.0, 87.0)
- added J1: ~, Connector_PinSocket_2.54mm:PinSocket_1x03_P2.54mm_Horizontal, B.Cu at (185.5, 42.5)
- added J1: ~, Connector_PinSocket_2.54mm:PinSocket_1x03_P2.54mm_Horizontal, B.Cu at (153.5, 98.5)
- added J1: ~, Connector_PinSocket_2.54mm:PinSocket_1x03_P2.54mm_Horizontal, B.Cu at (121.5, 70.5)
- added J1: ~, Connector_PinSocket_2.54mm:PinSocket_1x03_P2.54mm_Horizontal, B.Cu at (169.5, 70.5)
- added J1: ~, Connector_PinSocket_2.54mm:PinSocket_1x03_P2.54mm_Horizontal, B.Cu at (185.5, 98.5)
- added J1: ~, Connector_PinSocket_2.54mm:PinSocket_1x03_P2.54mm_Horizontal, B.Cu at (153.5, 70.5)
- added J1: ~, Connector_PinSocket_2.54mm:PinSocket_1x03_P2.54mm_Horizontal, B.Cu at (153.5, 42.5)
- added J1: ~, Connector_PinSocket_2.54mm:PinSocket_1x03_P2.54mm_Horizontal, B.Cu at (185.5, 70.5)
- added J1: ~, Connector_PinSocket_2.54mm:PinSocket_1x03_P2.54mm_Horizontal, B.Cu at (137.5, 70.5)
- added J1: ~, Connector_PinSocket_2.54mm:PinSocket_1x03_P2.54mm_Horizontal, B.Cu at (121.5, 98.5)
- added J1: ~, Connector_PinSocket_2.54mm:PinSocket_1x03_P2.54mm_Horizontal, B.Cu at (121.5, 42.5)
- added J1: ~, Connector_PinSocket_2.54mm:PinSocket_1x03_P2.54mm_Horizontal, B.Cu at (169.5, 42.5)
- added J1: ~, Connector_PinSocket_2.54mm:PinSocket_1x03_P2.54mm_Horizontal, B.Cu at (105.5, 98.5)
- added J1: ~, Connector_PinSocket_2.54mm:PinSocket_1x03_P2.54mm_Horizontal, B.Cu at (169.5, 98.5)
- added J1: ~, Connector_PinSocket_2.54mm:PinSocket_1x03_P2.54mm_Horizontal, B.Cu at (105.5, 70.5)
- added J1: ~, Connector_PinSocket_2.54mm:PinSocket_1x03_P2.54mm_Horizontal, B.Cu at (105.5, 42.5)
- added J1: ~, Connector_PinSocket_2.54mm:PinSocket_1x03_P2.54mm_Horizontal, B.Cu at (137.5, 42.5)
- added J1: ~, Connector_PinSocket_2.54mm:PinSocket_1x03_P2.54mm_Horizontal, B.Cu at (137.5, 98.5)
- added J3: USB_C_Receptacle_PowerOnly_6P, Connector_USB:USB_C_Receptacle_GCT_USB4125-xx-x_6P_TopMnt_Horizontal, F.Cu at (161.5, 68.0)
- added J3: USB_C_Receptacle_PowerOnly_6P, Connector_USB:USB_C_Receptacle_GCT_USB4125-xx-x_6P_TopMnt_Horizontal, F.Cu at (161.5, 40.0)
- added J3: USB_C_Receptacle_PowerOnly_6P, Connector_USB:USB_C_Receptacle_GCT_USB4125-xx-x_6P_TopMnt_Horizontal, F.Cu at (145.5, 68.0)
- added J3: USB_C_Receptacle_PowerOnly_6P, Connector_USB:USB_C_Receptacle_GCT_USB4125-xx-x_6P_TopMnt_Horizontal, F.Cu at (129.5, 68.0)
- added J3: USB_C_Receptacle_PowerOnly_6P, Connector_USB:USB_C_Receptacle_GCT_USB4125-xx-x_6P_TopMnt_Horizontal, F.Cu at (113.5, 40.0)
- added J3: USB_C_Receptacle_PowerOnly_6P, Connector_USB:USB_C_Receptacle_GCT_USB4125-xx-x_6P_TopMnt_Horizontal, F.Cu at (113.5, 68.0)
- added J3: USB_C_Receptacle_PowerOnly_6P, Connector_USB:USB_C_Receptacle_GCT_USB4125-xx-x_6P_TopMnt_Horizontal, F.Cu at (129.5, 40.0)
- added J3: USB_C_Receptacle_PowerOnly_6P, Connector_USB:USB_C_Receptacle_GCT_USB4125-xx-x_6P_TopMnt_Horizontal, F.Cu at (193.5, 68.0)
- added J3: USB_C_Receptacle_PowerOnly_6P, Connector_USB:USB_C_Receptacle_GCT_USB4125-xx-x_6P_TopMnt_Horizontal, F.Cu at (145.5, 40.0)
- added J3: USB_C_Receptacle_PowerOnly_6P, Connector_USB:USB_C_Receptacle_GCT_USB4125-xx-x_6P_TopMnt_Horizontal, F.Cu at (113.5, 96.0)
- added J3: USB_C_Receptacle_PowerOnly_6P, Connector_USB:USB_C_Receptacle_GCT_USB4125-xx-x_6P_TopMnt_Horizontal, F.Cu at (161.5, 96.0)
- added J3: USB_C_Receptacle_PowerOnly_6P, Connector_USB:USB_C_Receptacle_GCT_USB4125-xx-x_6P_TopMnt_Horizontal, F.Cu at (193.5, 40.0)
- added J3: USB_C_Receptacle_PowerOnly_6P, Connector_USB:USB_C_Receptacle_GCT_USB4125-xx-x_6P_TopMnt_Horizontal, F.Cu at (177.5, 96.0)
- added J3: USB_C_Receptacle_PowerOnly_6P, Connector_USB:USB_C_Receptacle_GCT_USB4125-xx-x_6P_TopMnt_Horizontal, F.Cu at (177.5, 68.0)
- added J3: USB_C_Receptacle_PowerOnly_6P, Connector_USB:USB_C_Receptacle_GCT_USB4125-xx-x_6P_TopMnt_Horizontal, F.Cu at (129.5, 96.0)
- added J3: USB_C_Receptacle_PowerOnly_6P, Connector_USB:USB_C_Receptacle_GCT_USB4125-xx-x_6P_TopMnt_Horizontal, F.Cu at (145.5, 96.0)
- added J3: USB_C_Receptacle_PowerOnly_6P, Connector_USB:USB_C_Receptacle_GCT_USB4125-xx-x_6P_TopMnt_Horizontal, F.Cu at (177.5, 40.0)
- added J3: USB_C_Receptacle_PowerOnly_6P, Connector_USB:USB_C_Receptacle_GCT_USB4125-xx-x_6P_TopMnt_Horizontal, F.Cu at (193.5, 96.0)
- added R1: 10k, Resistor_SMD:R_0805_2012Metric_Pad1.20x1.40mm_HandSolder, B.Cu at (188.0, 98.5)
- added R1: 10k, Resistor_SMD:R_0805_2012Metric_Pad1.20x1.40mm_HandSolder, B.Cu at (172.0, 98.5)
- added R1: 10k, Resistor_SMD:R_0805_2012Metric_Pad1.20x1.40mm_HandSolder, B.Cu at (156.0, 70.5)
- added R1: 10k, Resistor_SMD:R_0805_2012Metric_Pad1.20x1.40mm_HandSolder, B.Cu at (156.0, 98.5)
- added R1: 10k, Resistor_SMD:R_0805_2012Metric_Pad1.20x1.40mm_HandSolder, B.Cu at (188.0, 42.5)
- added R1: 10k, Resistor_SMD:R_0805_2012Metric_Pad1.20x1.40mm_HandSolder, B.Cu at (124.0, 70.5)
- added R1: 10k, Resistor_SMD:R_0805_2012Metric_Pad1.20x1.40mm_HandSolder, B.Cu at (108.0, 98.5)
- added R1: 10k, Resistor_SMD:R_0805_2012Metric_Pad1.20x1.40mm_HandSolder, B.Cu at (172.0, 42.5)
- added R1: 10k, Resistor_SMD:R_0805_2012Metric_Pad1.20x1.40mm_HandSolder, B.Cu at (172.0, 70.5)
- added R1: 10k, Resistor_SMD:R_0805_2012Metric_Pad1.20x1.40mm_HandSolder, B.Cu at (188.0, 70.5)
- added R1: 10k, Resistor_SMD:R_0805_2012Metric_Pad1.20x1.40mm_HandSolder, B.Cu at (108.0, 42.5)
- added R1: 10k, Resistor_SMD:R_0805_2012Metric_Pad1.20x1.40mm_HandSolder, B.Cu at (156.0, 42.5)
- added R1: 10k, Resistor_SMD:R_0805_2012Metric_Pad1.20x1.40mm_HandSolder, B.Cu at (140.0, 70.5)
- added R1: 10k, Resistor_SMD:R_0805_2012Metric_Pad1.20x1.40mm_HandSolder, B.Cu at (124.0, 98.5)
- added R1: 10k, Resistor_SMD:R_0805_2012Metric_Pad1.20x1.40mm_HandSolder, B.Cu at (140.0, 98.5)
- added R1: 10k, Resistor_SMD:R_0805_2012Metric_Pad1.20x1.40mm_HandSolder, B.Cu at (124.0, 42.5)
- added R1: 10k, Resistor_SMD:R_0805_2012Metric_Pad1.20x1.40mm_HandSolder, B.Cu at (140.0, 42.5)
- added R1: 10k, Resistor_SMD:R_0805_2012Metric_Pad1.20x1.40mm_HandSolder, B.Cu at (108.0, 70.5)
- added R2: 120, Resistor_SMD:R_0805_2012Metric_Pad1.20x1.40mm_HandSolder, B.Cu at (140.0, 38.5)
- added R2: 120, Resistor_SMD:R_0805_2012Metric_Pad1.20x1.40mm_HandSolder, B.Cu at (124.0, 66.5)
- added R2: 120, Resistor_SMD:R_0805_2012Metric_Pad1.20x1.40mm_HandSolder, B.Cu at (108.0, 38.5)
- added R2: 120, Resistor_SMD:R_0805_2012Metric_Pad1.20x1.40mm_HandSolder, B.Cu at (172.0, 94.5)
- added R2: 120, Resistor_SMD:R_0805_2012Metric_Pad1.20x1.40mm_HandSolder, B.Cu at (108.0, 66.5)
- added R2: 120, Resistor_SMD:R_0805_2012Metric_Pad1.20x1.40mm_HandSolder, B.Cu at (172.0, 38.5)
- added R2: 120, Resistor_SMD:R_0805_2012Metric_Pad1.20x1.40mm_HandSolder, B.Cu at (124.0, 38.5)
- added R2: 120, Resistor_SMD:R_0805_2012Metric_Pad1.20x1.40mm_HandSolder, B.Cu at (140.0, 94.5)
- added R2: 120, Resistor_SMD:R_0805_2012Metric_Pad1.20x1.40mm_HandSolder, B.Cu at (172.0, 66.5)
- added R2: 120, Resistor_SMD:R_0805_2012Metric_Pad1.20x1.40mm_HandSolder, B.Cu at (124.0, 94.5)
- added R2: 120, Resistor_SMD:R_0805_2012Metric_Pad1.20x1.40mm_HandSolder, B.Cu at (156.0, 66.5)
- added R2: 120, Resistor_SMD:R_0805_2012Metric_Pad1.20x1.40mm_HandSolder, B.Cu at (188.0, 38.5)
- added R2: 120, Resistor_SMD:R_0805_2012Metric_Pad1.20x1.40mm_HandSolder, B.Cu at (156.0, 38.5)
- added R2: 120, Resistor_SMD:R_0805_2012Metric_Pad1.20x1.40mm_HandSolder, B.Cu at (188.0, 66.5)
- added R2: 120, Resistor_SMD:R_0805_2012Metric_Pad1.20x1.40mm_HandSolder, B.Cu at (156.0, 94.5)
- added R2: 120, Resistor_SMD:R_0805_2012Metric_Pad1.20x1.40mm_HandSolder, B.Cu at (140.0, 66.5)
- added R2: 120, Resistor_SMD:R_0805_2012Metric_Pad1.20x1.40mm_HandSolder, B.Cu at (188.0, 94.5)
- added R2: 120, Resistor_SMD:R_0805_2012Metric_Pad1.20x1.40mm_HandSolder, B.Cu at (108.0, 94.5)
- added R3: 10k, Resistor_SMD:R_0805_2012Metric_Pad1.20x1.40mm_HandSolder, F.Cu at (124.0, 90.0)
- added R3: 10k, Resistor_SMD:R_0805_2012Metric_Pad1.20x1.40mm_HandSolder, F.Cu at (172.0, 90.0)
- added R3: 10k, Resistor_SMD:R_0805_2012Metric_Pad1.20x1.40mm_HandSolder, F.Cu at (108.0, 34.0)
- added R3: 10k, Resistor_SMD:R_0805_2012Metric_Pad1.20x1.40mm_HandSolder, F.Cu at (124.0, 62.0)
- added R3: 10k, Resistor_SMD:R_0805_2012Metric_Pad1.20x1.40mm_HandSolder, F.Cu at (156.0, 34.0)
- added R3: 10k, Resistor_SMD:R_0805_2012Metric_Pad1.20x1.40mm_HandSolder, F.Cu at (188.0, 90.0)
- added R3: 10k, Resistor_SMD:R_0805_2012Metric_Pad1.20x1.40mm_HandSolder, F.Cu at (172.0, 34.0)
- added R3: 10k, Resistor_SMD:R_0805_2012Metric_Pad1.20x1.40mm_HandSolder, F.Cu at (156.0, 90.0)
- added R3: 10k, Resistor_SMD:R_0805_2012Metric_Pad1.20x1.40mm_HandSolder, F.Cu at (156.0, 62.0)
- added R3: 10k, Resistor_SMD:R_0805_2012Metric_Pad1.20x1.40mm_HandSolder, F.Cu at (108.0, 90.0)
- added R3: 10k, Resistor_SMD:R_0805_2012Metric_Pad1.20x1.40mm_HandSolder, F.Cu at (124.0, 34.0)
- added R3: 10k, Resistor_SMD:R_0805_2012Metric_Pad1.20x1.40mm_HandSolder, F.Cu at (172.0, 62.0)
- added R3: 10k, Resistor_SMD:R_0805_2012Metric_Pad1.20x1.40mm_HandSolder, F.Cu at (108.0, 62.0)
- added R3: 10k, Resistor_SMD:R_0805_2012Metric_Pad1.20x1.40mm_HandSolder, F.Cu at (140.0, 62.0)
- added R3: 10k, Resistor_SMD:R_0805_2012Metric_Pad1.20x1.40mm_HandSolder, F.Cu at (140.0, 34.0)
- added R3: 10k, Resistor_SMD:R_0805_2012Metric_Pad1.20x1.40mm_HandSolder, F.Cu at (188.0, 34.0)
- added R3: 10k, Resistor_SMD:R_0805_2012Metric_Pad1.20x1.40mm_HandSolder, F.Cu at (140.0, 90.0)
- added R3: 10k, Resistor_SMD:R_0805_2012Metric_Pad1.20x1.40mm_HandSolder, F.Cu at (188.0, 62.0)
- added R4: 10k, Resistor_SMD:R_0805_2012Metric_Pad1.20x1.40mm_HandSolder, F.Cu at (169.5, 90.0)
- added R4: 10k, Resistor_SMD:R_0805_2012Metric_Pad1.20x1.40mm_HandSolder, F.Cu at (137.5, 90.0)
- added R4: 10k, Resistor_SMD:R_0805_2012Metric_Pad1.20x1.40mm_HandSolder, F.Cu at (185.5, 34.0)
- added R4: 10k, Resistor_SMD:R_0805_2012Metric_Pad1.20x1.40mm_HandSolder, F.Cu at (153.5, 34.0)
- added R4: 10k, Resistor_SMD:R_0805_2012Metric_Pad1.20x1.40mm_HandSolder, F.Cu at (121.5, 34.0)
- added R4: 10k, Resistor_SMD:R_0805_2012Metric_Pad1.20x1.40mm_HandSolder, F.Cu at (169.5, 34.0)
- added R4: 10k, Resistor_SMD:R_0805_2012Metric_Pad1.20x1.40mm_HandSolder, F.Cu at (137.5, 62.0)
- added R4: 10k, Resistor_SMD:R_0805_2012Metric_Pad1.20x1.40mm_HandSolder, F.Cu at (105.5, 90.0)
- added R4: 10k, Resistor_SMD:R_0805_2012Metric_Pad1.20x1.40mm_HandSolder, F.Cu at (137.5, 34.0)
- added R4: 10k, Resistor_SMD:R_0805_2012Metric_Pad1.20x1.40mm_HandSolder, F.Cu at (105.5, 34.0)
- added R4: 10k, Resistor_SMD:R_0805_2012Metric_Pad1.20x1.40mm_HandSolder, F.Cu at (185.5, 90.0)
- added R4: 10k, Resistor_SMD:R_0805_2012Metric_Pad1.20x1.40mm_HandSolder, F.Cu at (153.5, 90.0)
- added R4: 10k, Resistor_SMD:R_0805_2012Metric_Pad1.20x1.40mm_HandSolder, F.Cu at (153.5, 62.0)
- added R4: 10k, Resistor_SMD:R_0805_2012Metric_Pad1.20x1.40mm_HandSolder, F.Cu at (121.5, 62.0)
- added R4: 10k, Resistor_SMD:R_0805_2012Metric_Pad1.20x1.40mm_HandSolder, F.Cu at (121.5, 90.0)
- added R4: 10k, Resistor_SMD:R_0805_2012Metric_Pad1.20x1.40mm_HandSolder, F.Cu at (105.5, 62.0)
- added R4: 10k, Resistor_SMD:R_0805_2012Metric_Pad1.20x1.40mm_HandSolder, F.Cu at (185.5, 62.0)
- added R4: 10k, Resistor_SMD:R_0805_2012Metric_Pad1.20x1.40mm_HandSolder, F.Cu at (169.5, 62.0)
- added R5: 5.1k, Resistor_SMD:R_0805_2012Metric_Pad1.20x1.40mm_HandSolder, B.Cu at (127.5, 97.0)
- added R5: 5.1k, Resistor_SMD:R_0805_2012Metric_Pad1.20x1.40mm_HandSolder, B.Cu at (191.5, 41.0)
- added R5: 5.1k, Resistor_SMD:R_0805_2012Metric_Pad1.20x1.40mm_HandSolder, B.Cu at (159.5, 41.0)
- added R5: 5.1k, Resistor_SMD:R_0805_2012Metric_Pad1.20x1.40mm_HandSolder, B.Cu at (143.5, 97.0)
- added R5: 5.1k, Resistor_SMD:R_0805_2012Metric_Pad1.20x1.40mm_HandSolder, B.Cu at (191.5, 69.0)
- added R5: 5.1k, Resistor_SMD:R_0805_2012Metric_Pad1.20x1.40mm_HandSolder, B.Cu at (111.5, 97.0)
- added R5: 5.1k, Resistor_SMD:R_0805_2012Metric_Pad1.20x1.40mm_HandSolder, B.Cu at (143.5, 69.0)
- added R5: 5.1k, Resistor_SMD:R_0805_2012Metric_Pad1.20x1.40mm_HandSolder, B.Cu at (175.5, 97.0)
- added R5: 5.1k, Resistor_SMD:R_0805_2012Metric_Pad1.20x1.40mm_HandSolder, B.Cu at (175.5, 41.0)
- added R5: 5.1k, Resistor_SMD:R_0805_2012Metric_Pad1.20x1.40mm_HandSolder, B.Cu at (127.5, 41.0)
- added R5: 5.1k, Resistor_SMD:R_0805_2012Metric_Pad1.20x1.40mm_HandSolder, B.Cu at (175.5, 69.0)
- added R5: 5.1k, Resistor_SMD:R_0805_2012Metric_Pad1.20x1.40mm_HandSolder, B.Cu at (159.5, 69.0)
- added R5: 5.1k, Resistor_SMD:R_0805_2012Metric_Pad1.20x1.40mm_HandSolder, B.Cu at (111.5, 41.0)
- added R5: 5.1k, Resistor_SMD:R_0805_2012Metric_Pad1.20x1.40mm_HandSolder, B.Cu at (159.5, 97.0)
- added R5: 5.1k, Resistor_SMD:R_0805_2012Metric_Pad1.20x1.40mm_HandSolder, B.Cu at (127.5, 69.0)
- added R5: 5.1k, Resistor_SMD:R_0805_2012Metric_Pad1.20x1.40mm_HandSolder, B.Cu at (143.5, 41.0)
- added R5: 5.1k, Resistor_SMD:R_0805_2012Metric_Pad1.20x1.40mm_HandSolder, B.Cu at (191.5, 97.0)
- added R5: 5.1k, Resistor_SMD:R_0805_2012Metric_Pad1.20x1.40mm_HandSolder, B.Cu at (111.5, 69.0)
- added R6: 5.1k, Resistor_SMD:R_0805_2012Metric_Pad1.20x1.40mm_HandSolder, B.Cu at (175.5, 67.0)
- added R6: 5.1k, Resistor_SMD:R_0805_2012Metric_Pad1.20x1.40mm_HandSolder, B.Cu at (127.5, 39.0)
- added R6: 5.1k, Resistor_SMD:R_0805_2012Metric_Pad1.20x1.40mm_HandSolder, B.Cu at (191.5, 67.0)
- added R6: 5.1k, Resistor_SMD:R_0805_2012Metric_Pad1.20x1.40mm_HandSolder, B.Cu at (159.5, 95.0)
- added R6: 5.1k, Resistor_SMD:R_0805_2012Metric_Pad1.20x1.40mm_HandSolder, B.Cu at (127.5, 67.0)
- added R6: 5.1k, Resistor_SMD:R_0805_2012Metric_Pad1.20x1.40mm_HandSolder, B.Cu at (191.5, 39.0)
- added R6: 5.1k, Resistor_SMD:R_0805_2012Metric_Pad1.20x1.40mm_HandSolder, B.Cu at (111.5, 95.0)
- added R6: 5.1k, Resistor_SMD:R_0805_2012Metric_Pad1.20x1.40mm_HandSolder, B.Cu at (175.5, 39.0)
- added R6: 5.1k, Resistor_SMD:R_0805_2012Metric_Pad1.20x1.40mm_HandSolder, B.Cu at (127.5, 95.0)
- added R6: 5.1k, Resistor_SMD:R_0805_2012Metric_Pad1.20x1.40mm_HandSolder, B.Cu at (143.5, 95.0)
- added R6: 5.1k, Resistor_SMD:R_0805_2012Metric_Pad1.20x1.40mm_HandSolder, B.Cu at (143.5, 67.0)
- added R6: 5.1k, Resistor_SMD:R_0805_2012Metric_Pad1.20x1.40mm_HandSolder, B.Cu at (111.5, 67.0)
- added R6: 5.1k, Resistor_SMD:R_0805_2012Metric_Pad1.20x1.40mm_HandSolder, B.Cu at (159.5, 67.0)
- added R6: 5.1k, Resistor_SMD:R_0805_2012Metric_Pad1.20x1.40mm_HandSolder, B.Cu at (159.5, 39.0)
- added R6: 5.1k, Resistor_SMD:R_0805_2012Metric_Pad1.20x1.40mm_HandSolder, B.Cu at (191.5, 95.0)
- added R6: 5.1k, Resistor_SMD:R_0805_2012Metric_Pad1.20x1.40mm_HandSolder, B.Cu at (111.5, 39.0)
- added R6: 5.1k, Resistor_SMD:R_0805_2012Metric_Pad1.20x1.40mm_HandSolder, B.Cu at (175.5, 95.0)
- added R6: 5.1k, Resistor_SMD:R_0805_2012Metric_Pad1.20x1.40mm_HandSolder, B.Cu at (143.5, 39.0)
- U2 (x18): moved to B.Cu
- moved KiKit_MB_3_1 25.2 mm to (110.0, 52.5)
- moved KiKit_MB_3_4 25.2 mm to (107.0, 52.5)
- moved KiKit_MB_4_1 25.2 mm to (107.0, 27.5)
- moved KiKit_MB_4_4 25.2 mm to (110.0, 27.5)
- moved KiKit_MB_35_1 25.2 mm to (110.0, 80.5)
- moved KiKit_MB_35_4 25.2 mm to (107.0, 80.5)
- moved KiKit_MB_36_1 25.2 mm to (107.0, 55.5)
- moved KiKit_MB_36_4 25.2 mm to (110.0, 55.5)
- moved KiKit_MB_67_1 25.2 mm to (110.0, 108.5)
- moved KiKit_MB_67_4 25.2 mm to (107.0, 108.5)
- moved KiKit_MB_68_1 25.2 mm to (107.0, 83.5)
- moved KiKit_MB_68_4 25.2 mm to (110.0, 83.5)
- moved KiKit_MB_3_2 25.0 mm to (109.0, 52.5)
- moved KiKit_MB_3_3 25.0 mm to (108.0, 52.5)
- moved KiKit_MB_4_2 25.0 mm to (108.0, 27.5)
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Connections:
- U1_ pad 1: (no net) -> Board_17-unconnected-(U1-URXD-Pad8)
- U1_ pad 8: (no net) -> Board_17-unconnected-(U1-UTXD-Pad1)
- U1_ pad 1: (no net) -> Board_4-unconnected-(U1-URXD-Pad8)
- U1_ pad 8: (no net) -> Board_4-unconnected-(U1-UTXD-Pad1)
- U1_ pad 1: (no net) -> Board_2-unconnected-(U1-URXD-Pad8)
- U1_ pad 8: (no net) -> Board_2-unconnected-(U1-UTXD-Pad1)
- U1_ pad 1: (no net) -> Board_6-unconnected-(U1-URXD-Pad8)
- U1_ pad 8: (no net) -> Board_6-unconnected-(U1-UTXD-Pad1)
- U1_ pad 1: (no net) -> Board_10-unconnected-(U1-URXD-Pad8)
- U1_ pad 8: (no net) -> Board_10-unconnected-(U1-UTXD-Pad1)
- U1_ pad 1: (no net) -> Board_0-unconnected-(U1-URXD-Pad8)
- U1_ pad 8: (no net) -> Board_0-unconnected-(U1-UTXD-Pad1)
- U1_ pad 1: (no net) -> Board_15-unconnected-(U1-URXD-Pad8)
- U1_ pad 8: (no net) -> Board_15-unconnected-(U1-UTXD-Pad1)
- U1_ pad 1: (no net) -> Board_3-unconnected-(U1-URXD-Pad8)
- U1_ pad 8: (no net) -> Board_3-unconnected-(U1-UTXD-Pad1)
- U1_ pad 1: (no net) -> Board_12-unconnected-(U1-URXD-Pad8)
- U1_ pad 8: (no net) -> Board_12-unconnected-(U1-UTXD-Pad1)
- U1_ pad 1: (no net) -> Board_9-unconnected-(U1-URXD-Pad8)
- U1_ pad 8: (no net) -> Board_9-unconnected-(U1-UTXD-Pad1)
- U1_ pad 1: (no net) -> Board_13-unconnected-(U1-URXD-Pad8)
- U1_ pad 8: (no net) -> Board_13-unconnected-(U1-UTXD-Pad1)
- U1_ pad 1: (no net) -> Board_11-unconnected-(U1-URXD-Pad8)
- U1_ pad 8: (no net) -> Board_11-unconnected-(U1-UTXD-Pad1)
- U1_ pad 1: (no net) -> Board_14-unconnected-(U1-URXD-Pad8)
- U1_ pad 8: (no net) -> Board_14-unconnected-(U1-UTXD-Pad1)
- U1_ pad 1: (no net) -> Board_5-unconnected-(U1-URXD-Pad8)
- U1_ pad 8: (no net) -> Board_5-unconnected-(U1-UTXD-Pad1)
- U1_ pad 1: (no net) -> Board_7-unconnected-(U1-URXD-Pad8)
- U1_ pad 8: (no net) -> Board_7-unconnected-(U1-UTXD-Pad1)
- U1_ pad 1: (no net) -> Board_1-unconnected-(U1-URXD-Pad8)
- U1_ pad 8: (no net) -> Board_1-unconnected-(U1-UTXD-Pad1)
- U1_ pad 1: (no net) -> Board_16-unconnected-(U1-URXD-Pad8)
- U1_ pad 8: (no net) -> Board_16-unconnected-(U1-UTXD-Pad1)
- U1_ pad 1: (no net) -> Board_8-unconnected-(U1-URXD-Pad8)
- U1_ pad 8: (no net) -> Board_8-unconnected-(U1-UTXD-Pad1)
Routing:
- net Board_9-GND: track 3.53 -> 15.2 mm
- net Board_8-GND: track 3.53 -> 15.2 mm
- net Board_17-GND: track 3.53 -> 15.2 mm
- net Board_16-GND: track 3.53 -> 15.2 mm
- net Board_15-GND: track 3.53 -> 15.2 mm
- net Board_14-GND: track 3.53 -> 15.2 mm
- net Board_11-GND: track 3.53 -> 15.2 mm
- net Board_10-GND: track 3.53 -> 15.2 mm
- net Board_5-GND: track 3.53 -> 15.2 mm
- net Board_4-GND: track 3.53 -> 15.2 mm
- net Board_3-GND: track 3.53 -> 15.2 mm
- net Board_2-GND: track 3.53 -> 15.2 mm
- net Board_7-GND: track 3.53 -> 15.2 mm
- net Board_6-GND: track 3.53 -> 15.2 mm
- net Board_13-GND: track 3.53 -> 15.2 mm
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- added copper zone on B.Cu, net Board_0-GND
- added copper zone on F.Cu, net Board_0-GND
- added copper zone on B.Cu, net Board_1-GND
- added copper zone on F.Cu, net Board_1-GND
- added copper zone on B.Cu, net Board_10-GND
- added copper zone on F.Cu, net Board_10-GND
- added copper zone on B.Cu, net Board_11-GND
- added copper zone on F.Cu, net Board_11-GND
- added copper zone on B.Cu, net Board_12-GND
- added copper zone on F.Cu, net Board_12-GND
- added copper zone on B.Cu, net Board_13-GND
- added copper zone on F.Cu, net Board_13-GND
- added copper zone on B.Cu, net Board_14-GND
- added copper zone on F.Cu, net Board_14-GND
- added copper zone on B.Cu, net Board_15-GND
- added copper zone on F.Cu, net Board_15-GND
- added copper zone on B.Cu, net Board_16-GND
- added copper zone on F.Cu, net Board_16-GND
- added copper zone on B.Cu, net Board_17-GND
- added copper zone on F.Cu, net Board_17-GND
- added copper zone on B.Cu, net Board_2-GND
- added copper zone on F.Cu, net Board_2-GND
- added copper zone on B.Cu, net Board_3-GND
- added copper zone on F.Cu, net Board_3-GND
- added copper zone on B.Cu, net Board_4-GND
- added copper zone on F.Cu, net Board_4-GND
- added copper zone on B.Cu, net Board_5-GND
- added copper zone on F.Cu, net Board_5-GND
- added copper zone on B.Cu, net Board_6-GND
- added copper zone on F.Cu, net Board_6-GND
- added copper zone on B.Cu, net Board_7-GND
- added copper zone on F.Cu, net Board_7-GND
- added copper zone on B.Cu, net Board_8-GND
- added copper zone on F.Cu, net Board_8-GND
- added copper zone on B.Cu, net Board_9-GND
- added copper zone on F.Cu, net Board_9-GND
Other:
- outline, holes or cut-outs redrawn
